File: hardware/schematic/adc-conditioner.kicad_sch (KiCad schematic)
At the start: 42 parts

Commit message: refactor structure
Parts:
- gave numbers to parts that had none: 36

Commit message: schematic finished
Parts:
- added C17: 100nF,100V, symbol Device:C
- added R30: 2M, Resistor_SMD:R_0805_2012Metric_Pad1.20x1.40mm_HandSolder, symbol Device:R
- added R31: 100k, Resistor_SMD:R_0805_2012Metric_Pad1.20x1.40mm_HandSolder, symbol Device:R
- renumbered C14 to C18, C15 to C19, C16 to C20, C17 to C21, C18 to C22, C19 to C23, C20 to C24, C21 to C25, C22 to C26, C23 to C27, C24 to C28, R31 to R32, R32 to R33, R33 to R34, R34 to R35, R35 to R36, R36 to R37, R37 to R38, R38 to R39, R39 to R40, R40 to R41, R41 to R42, R42 to R43, R43 to R44, R44 to R45, R45 to R46, R46 to R47, R47 to R48, R48 to R49
Connections:
- net at U6.5 (+): now also C17.1, R30.2, R31.1
- net VOLT_TOTAL: now reaches U6.6 (-)
- net VOLT_TOTAL: now also U6.7
- net COND_A_CUR renamed CUR_A
- net COND_B_CUR renamed CUR_B
- net COND_C_CUR renamed CUR_C
- net COND_TOTAL_CUR renamed CUR_TOTAL
- net CURRENT_A_HIGH renamed CUR_A_H
- net CURRENT_A_LOW renamed CUR_A_L
- net CURRENT_B_HIGH renamed CUR­_B_H
- net CURRENT_B_LOW renamed CUR_B_L
- net CURRENT_C_HIGH renamed CUR_C_H
- net CURRENT_C_LOW renamed CUR_C_L
- net CURRENT_TOTAL_HIGH renamed CUR_TOTAL_H
- net CURRENT_TOTAL_LOW renamed CUR_TOTAL_L
- new net GNDPWR: C17.2, R31.2
- new net Vdrive: R30.1
Other:
- moved on the sheet: U6B

Commit message: pcb improvements
Parts:
- C16: renamed from C17; footprint (none) -> Capacitor_SMD:C_0805_2012Metric_Pad1.18x1.45mm_HandSolder
- C17: renamed from C18; footprint (none) -> Capacitor_SMD:C_0805_2012Metric_Pad1.18x1.45mm_HandSolder
- C18: renamed from C19; footprint (none) -> Capacitor_SMD:C_0805_2012Metric_Pad1.18x1.45mm_HandSolder
- C19: renamed from C20; footprint (none) -> Capacitor_SMD:C_0805_2012Metric_Pad1.18x1.45mm_HandSolder
- C20: renamed from C21; footprint (none) -> Capacitor_SMD:C_0805_2012Metric_Pad1.18x1.45mm_HandSolder
- C21: renamed from C22; footprint (none) -> Capacitor_SMD:C_0805_2012Metric_Pad1.18x1.45mm_HandSolder
- C22: renamed from C23; footprint (none) -> Capacitor_SMD:C_0805_2012Metric_Pad1.18x1.45mm_HandSolder
- C23: renamed from C24; footprint (none) -> Capacitor_SMD:C_0805_2012Metric_Pad1.18x1.45mm_HandSolder
- C24: renamed from C25; footprint (none) -> Capacitor_SMD:C_0805_2012Metric_Pad1.18x1.45mm_HandSolder
- C25: renamed from C26; footprint (none) -> Capacitor_SMD:C_0805_2012Metric_Pad1.18x1.45mm_HandSolder
- C26: renamed from C27; footprint (none) -> Capacitor_SMD:C_0805_2012Metric_Pad1.18x1.45mm_HandSolder
- C27: renamed from C28; footprint (none) -> Capacitor_SMD:C_0805_2012Metric_Pad1.18x1.45mm_HandSolder
- renumbered R30 to R29, R31 to R30, R32 to R31, R33 to R32, R34 to R33, R35 to R34, R36 to R35, R37 to R36, R38 to R37, R39 to R38, R40 to R39, R41 to R40, R42 to R41, R43 to R42, R44 to R43, R45 to R44, R46 to R45, R47 to R46, R48 to R47, R49 to R48
Connections:
- net CUR_A_H renamed CUR_A_P
- net CUR_A_L renamed CUR_A_N
- net CUR_B_L renamed CUR_B_N
- net CUR_C_H renamed CUR_C_P
- net CUR_C_L renamed CUR_C_N
- net CUR_TOTAL_H renamed CUR_TOTAL_P
- net CUR_TOTAL_L renamed CUR_TOTAL_N
- net CUR­_B_H renamed CUR­_B_P
