File: hardware/schematic/can-bus.kicad_sch (KiCad schematic)
At the start: 1 part, among them U1 SN65HVD230

Commit message: refactor structure
Parts:
- renumbered U1 to U7
Changed lines of the file:
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@@
 		(dnp no)
 		(fields_autoplaced yes)
-		(property "Reference" "U1"
+		(property "Reference" "U7"
 			(at 146.9233 73.66 0)
 			(show_name no)
@@
 			(project "e-foc"
 				(path "/34e5c7b2-bc7d-4136-97dd-86505a14228c/deaffcfb-90c2-4afd-9218-7765e99e9a8e"
-					(reference "U1")
+					(reference "U7")
 					(unit 1)
 				)

Commit message: schematic finished
Parts:
- added C29, C30: 100nF,16V,X7R, symbol Device:C
- added C31: 4.7nF, symbol Device:C
- added D7: NUP2105L, Package_TO_SOT_SMD:SOT-23W_Handsoldering, symbol Power_Protection:NUP2105L
- added J3: Screw_Terminal_01x02, TerminalBlock_TE-Connectivity:TerminalBlock_TE_282834-2_1x02_P2.54mm_Horizontal, symbol Connector:Screw_Terminal_01x02
- added R50: 0R, Resistor_SMD:R_0805_2012Metric_Pad1.20x1.40mm_HandSolder, symbol Device:R
- added R51, R52: 60R, Resistor_SMD:R_0805_2012Metric_Pad1.20x1.40mm_HandSolder, symbol Device:R
Connections:
- net CAN_TX: now reaches U7.1 (D)
- net GND: now reaches U7.2 (GND)
- net GND: now also C29.2, C30.2, C31.2, D7.3 (A), R50.2
- net +3.3V: now reaches U7.3 (VCC)
- net +3.3V: now also C30.1
- net CAN_RX: now reaches U7.4 (R)
- net at U7.5 (Vref): now also C29.1
- net at U7.6 (CANL): now also D7.2 (K), J3.2 (Pin_2), R52.2
- net at U7.7 (CANH): now also D7.1 (K), J3.1 (Pin_1), R51.1
- net at U7.8 (Rs): now also R50.1
- new net: C31.1, R51.2, R52.1
Other:
- moved on the sheet: U7

Commit message: pcb improvements
Parts:
- C28: renamed from C29; footprint (none) -> Capacitor_SMD:C_0805_2012Metric_Pad1.18x1.45mm_HandSolder
- C29: renamed from C30; footprint (none) -> Capacitor_SMD:C_0805_2012Metric_Pad1.18x1.45mm_HandSolder
- C30: renamed from C31; footprint (none) -> Capacitor_SMD:C_0805_2012Metric_Pad1.18x1.45mm_HandSolder
- renumbered D7 to D6, R50 to R49, R51 to R50, R52 to R51
Connections:
- net at J3.1 (Pin_1), R50.1, U7.7 (CANH): now also D6.2 (K); no longer D6.1 (K)
- net at J3.2 (Pin_2), R51.2, U7.6 (CANL): now also D6.1 (K); no longer D6.2 (K)
Changed lines of the file:
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@@
 	(paper "A4")
-	(junction
-		(at 213.36 92.71)
-		(diameter 0)
-		(color 0 0 0 0)
-	)
 	(junction
 		(at 199.39 93.98)
@@
 	)
 	(junction
-		(at 199.39 105.41)
+		(at 213.36 95.25)
 		(diameter 0)
 		(color 0 0 0 0)
 	)
 	(junction
-		(at 218.44 95.25)
+		(at 199.39 105.41)
 		(diameter 0)
 		(color 0 0 0 0)
@@
 		(color 0 0 0 0)
 	)
-	(wire
-		(pts
-			(xy 224.79 92.71) (xy 213.36 92.71)
+	(junction
+		(at 218.44 92.71)
+		(diameter 0)
+		(color 0 0 0 0)
+	)
+	(wire
+		(pts
+			(xy 207.01 92.71) (xy 218.44 92.71)
 		)
 		(stroke
@@
 	(wire
 		(pts
-			(xy 213.36 92.71) (xy 213.36 101.6)
+			(xy 213.36 95.25) (xy 213.36 101.6)
 		)
 		(stroke
@@
 	(wire
 		(pts
-			(xy 218.44 95.25) (xy 224.79 95.25)
-		)
-		(stroke
-			(width 0)
-			(type default)
-		)
-	)
-	(wire
-		(pts
-			(xy 207.01 95.25) (xy 218.44 95.25)
+			(xy 207.01 95.25) (xy 213.36 95.25)
 		)
 		(stroke
@@
 	(wire
 		(pts
+			(xy 218.44 92.71) (xy 224.79 92.71)
+		)
+		(stroke
+			(width 0)
+			(type default)
+		)
+	)
+	(wire
+		(pts
 			(xy 207.01 105.41) (xy 199.39 105.41)
 		)
@@
 	(wire
 		(pts
+			(xy 213.36 95.25) (xy 224.79 95.25)
+		)
+		(stroke
+			(width 0)
+			(type default)
+		)
+	)
+	(wire
+		(pts
 			(xy 151.13 95.25) (xy 163.83 95.25)
 		)
@@
 	(wire
 		(pts
-			(xy 218.44 101.6) (xy 218.44 95.25)
+			(xy 218.44 92.71) (xy 218.44 101.6)
 		)
 		(stroke
@@
 		(pts
 			(xy 207.01 82.55) (xy 199.39 82.55)
-		)
-		(stroke
-			(width 0)
-			(type default)
-		)
-	)
-	(wire
-		(pts
-			(xy 213.36 92.71) (xy 207.01 92.71)
 		)
 		(stroke
@@
 		(dnp no)
 		(fields_autoplaced yes)
-		(property "Reference" "#PWR052"
+		(property "Reference" "#PWR050"
 			(at 173.99 119.38 0)
 			(hide yes)
@@
 			(project "e-foc"
 				(path "/34e5c7b2-bc7d-4136-97dd-86505a14228c/deaffcfb-90c2-4afd-9218-7765e99e9a8e"
-					(reference "#PWR052")
+					(reference "#PWR050")
 					(unit 1)
 				)
@@
 		(dnp no)
 		(fields_autoplaced yes)
-		(property "Reference" "#PWR053"
+		(property "Reference" "#PWR051"
 			(at 185.42 66.04 0)
 			(hide yes)
@@
 			(project "e-foc"
 				(path "/34e5c7b2-bc7d-4136-97dd-86505a14228c/deaffcfb-90c2-4afd-9218-7765e99e9a8e"
-					(reference "#PWR053")
+					(reference "#PWR051")
 					(unit 1)
 				)
@@
 		(in_pos_files yes)
 		(dnp no)
-		(property "Reference" "R50"
+		(property "Reference" "R49"
 			(at 161.29 106.6799 0)
 			(show_name no)
@@
 			(project "e-foc"
 				(path "/34e5c7b2-bc7d-4136-97dd-86505a14228c/deaffcfb-90c2-4afd-9218-7765e99e9a8e"
-					(reference "R50")
+					(reference "R49")
 					(unit 1)
 				)
@@
 		(dnp no)
 		(fields_autoplaced yes)
-		(property "Reference" "D7"
+		(property "Reference" "D6"
 			(at 222.25 105.4099 0)
 			(show_name no)
@@
 			(project "e-foc"
 				(path "/34e5c7b2-bc7d-4136-97dd-86505a14228c/deaffcfb-90c2-4afd-9218-7765e99e9a8e"
-					(reference "D7")
+					(reference "D6")
 					(unit 1)
 				)
@@
 		(dnp no)
 		(fields_autoplaced yes)
-		(property "Reference" "#PWR051"
+		(property "Reference" "#PWR049"
 			(at 173.99 87.63 0)
 			(hide yes)
@@
 			(project "e-foc"
 				(path "/34e5c7b2-bc7d-4136-97dd-86505a14228c/deaffcfb-90c2-4afd-9218-7765e99e9a8e"
-					(reference "#PWR051")
+					(reference "#PWR049")
 					(unit 1)
 				)
@@
 		(dnp no)
 		(fields_autoplaced yes)
-		(property "Reference" "#PWR056"
+		(property "Reference" "#PWR054"
 			(at 215.9 119.38 0)
 			(hide yes)
@@
 			(project "e-foc"
 				(path "/34e5c7b2-bc7d-4136-97dd-86505a14228c/deaffcfb-90c2-4afd-9218-7765e99e9a8e"
-					(reference "#PWR056")
+					(reference "#PWR054")
 					(unit 1)
 				)
@@
 		(in_pos_files yes)
 		(dnp no)
-		(property "Reference" "C31"
+		(property "Reference" "C30"
 			(at 190.5 104.1399 0)
 			(show_name no)
@@
 			)
 		)
-		(property "Footprint" ""
+		(property "Footprint" "Capacitor_SMD:C_0805_2012Metric_Pad1.18x1.45mm_HandSolder"
 			(at 187.6552 109.22 0)
 			(hide yes)
@@
 			(project "e-foc"
 				(path "/34e5c7b2-bc7d-4136-97dd-86505a14228c/deaffcfb-90c2-4afd-9218-7765e99e9a8e"
-					(reference "C31")
+					(reference "C30")
 					(unit 1)
 				)
@@
 		(dnp no)
 		(fields_autoplaced yes)
-		(property "Reference" "#PWR055"
+		(property "Reference" "#PWR053"
 			(at 186.69 119.38 0)
 			(hide yes)
@@
 			(project "e-foc"
 				(path "/34e5c7b2-bc7d-4136-97dd-86505a14228c/deaffcfb-90c2-4afd-9218-7765e99e9a8e"
-					(reference "#PWR055")
+					(reference "#PWR053")
 					(unit 1)
 				)
@@
 		(dnp no)
 		(fields_autoplaced yes)
-		(property "Reference" "#PWR054"
+		(property "Reference" "#PWR052"
 			(at 185.42 78.74 0)
 			(hide yes)
@@
 			(project "e-foc"
 				(path "/34e5c7b2-bc7d-4136-97dd-86505a14228c/deaffcfb-90c2-4afd-9218-7765e99e9a8e"
-					(reference "#PWR054")
+					(reference "#PWR052")
 					(unit 1)
 				)
@@
 		(in_pos_files yes)
 		(dnp no)
-		(property "Reference" "C29"
+		(property "Reference" "C28"
 			(at 154.178 106.426 0)
 			(show_name no)
@@
 			)
 		)
-		(property "Footprint" ""
+		(property "Footprint" "Capacitor_SMD:C_0805_2012Metric_Pad1.18x1.45mm_HandSolder"
 			(at 152.0952 111.76 0)
 			(hide yes)
@@
 			(project "e-foc"
 				(path "/34e5c7b2-bc7d-4136-97dd-86505a14228c/deaffcfb-90c2-4afd-9218-7765e99e9a8e"
-					(reference "C29")
+					(reference "C28")
 					(unit 1)
 				)
@@
 		(in_pos_files yes)
 		(dnp no)
-		(property "Reference" "R52"
+		(property "Reference" "R51"
 			(at 201.93 97.7899 0)
 			(show_name no)
@@
 			(project "e-foc"
 				(path "/34e5c7b2-bc7d-4136-97dd-86505a14228c/deaffcfb-90c2-4afd-9218-7765e99e9a8e"
-					(reference "R52")
+					(reference "R51")
 					(unit 1)
 				)
@@
 		(dnp no)
 		(fields_autoplaced yes)
-		(property "Reference" "#PWR050"
+		(property "Reference" "#PWR048"
 			(at 158.75 119.38 0)
 			(hide yes)
@@
 			(project "e-foc"
 				(path "/34e5c7b2-bc7d-4136-97dd-86505a14228c/deaffcfb-90c2-4afd-9218-7765e99e9a8e"
-					(reference "#PWR050")
+					(reference "#PWR048")
 					(unit 1)
 				)
@@
 		(dnp no)
 		(fields_autoplaced yes)
-		(property "Reference" "#PWR049"
+		(property "Reference" "#PWR047"
 			(at 151.13 119.38 0)
 			(hide yes)
@@
 			(project "e-foc"
 				(path "/34e5c7b2-bc7d-4136-97dd-86505a14228c/deaffcfb-90c2-4afd-9218-7765e99e9a8e"
-					(reference "#PWR049")
+					(reference "#PWR047")
 					(unit 1)
 				)
@@
 		(in_pos_files yes)
 		(dnp no)
-		(property "Reference" "C30"
+		(property "Reference" "C29"
 			(at 189.23 66.0399 0)
 			(show_name no)
@@
 			)
 		)
-		(property "Footprint" ""
+		(property "Footprint" "Capacitor_SMD:C_0805_2012Metric_Pad1.18x1.45mm_HandSolder"
 			(at 186.3852 71.12 0)
 			(hide yes)
@@
 			(project "e-foc"
 				(path "/34e5c7b2-bc7d-4136-97dd-86505a14228c/deaffcfb-90c2-4afd-9218-7765e99e9a8e"
-					(reference "C30")
+					(reference "C29")
 					(unit 1)
 				)
@@
 		(in_pos_files yes)
 		(dnp no)
-		(property "Reference" "R51"
+		(property "Reference" "R50"
 			(at 201.93 87.6299 0)
 			(show_name no)
@@
 			(project "e-foc"
 				(path "/34e5c7b2-bc7d-4136-97dd-86505a14228c/deaffcfb-90c2-4afd-9218-7765e99e9a8e"
-					(reference "R51")
+					(reference "R50")
 					(unit 1)
 				)

Commit message: updates
Parts:
- removed J3: Screw_Terminal_01x02, TerminalBlock_TE-Connectivity:TerminalBlock_TE_282834-2_1x02_P2.54mm_Horizontal, symbol Connector:Screw_Terminal_01x02
- added J3: Screw_Terminal_01x03, TerminalBlock:TerminalBlock_Xinya_XY308-2.54-3P_1x03_P2.54mm_Horizontal, symbol Connector:Screw_Terminal_01x03
Connections:
- net GND: now also J3.2 (Pin_2)
- net at D6.1 (K), R51.2, U7.6 (CANL): now also J3.3 (Pin_3)
- net at D6.2 (K), R50.1, U7.7 (CANH): now also J3.1 (Pin_1)
Changed lines of the file:
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@@
 	)
 	(junction
-		(at 213.36 95.25)
+		(at 218.44 91.44)
 		(diameter 0)
 		(color 0 0 0 0)
@@
 	)
 	(junction
-		(at 218.44 92.71)
+		(at 213.36 96.52)
 		(diameter 0)
 		(color 0 0 0 0)
@@
 	(wire
 		(pts
-			(xy 207.01 92.71) (xy 218.44 92.71)
-		)
-		(stroke
-			(width 0)
-			(type default)
-		)
-	)
-	(wire
-		(pts
 			(xy 185.42 71.12) (xy 185.42 72.39)
 		)
@@
 	(wire
 		(pts
-			(xy 207.01 92.71) (xy 207.01 82.55)
-		)
-		(stroke
-			(width 0)
-			(type default)
-		)
-	)
-	(wire
-		(pts
-			(xy 213.36 95.25) (xy 213.36 101.6)
+			(xy 224.79 97.79) (xy 224.79 93.98)
 		)
 		(stroke
@@
 	(wire
 		(pts
-			(xy 207.01 95.25) (xy 213.36 95.25)
+			(xy 207.01 96.52) (xy 207.01 105.41)
 		)
 		(stroke
@@
 	(wire
 		(pts
-			(xy 207.01 95.25) (xy 207.01 105.41)
-		)
-		(stroke
-			(width 0)
-			(type default)
-		)
-	)
-	(wire
-		(pts
-			(xy 218.44 92.71) (xy 224.79 92.71)
+			(xy 224.79 93.98) (xy 227.33 93.98)
+		)
+		(stroke
+			(width 0)
+			(type default)
+		)
+	)
+	(wire
+		(pts
+			(xy 207.01 96.52) (xy 213.36 96.52)
 		)
 		(stroke
@@
 	(wire
 		(pts
-			(xy 213.36 95.25) (xy 224.79 95.25)
-		)
-		(stroke
-			(width 0)
-			(type default)
-		)
-	)
-	(wire
-		(pts
 			(xy 151.13 95.25) (xy 163.83 95.25)
 		)
@@
 	(wire
 		(pts
-			(xy 218.44 92.71) (xy 218.44 101.6)
+			(xy 207.01 91.44) (xy 218.44 91.44)
+		)
+		(stroke
+			(width 0)
+			(type default)
+		)
+	)
+	(wire
+		(pts
+			(xy 213.36 96.52) (xy 227.33 96.52)
+		)
+		(stroke
+			(width 0)
+			(type default)
+		)
+	)
+	(wire
+		(pts
+			(xy 218.44 91.44) (xy 227.33 91.44)
 		)
 		(stroke
@@
 	(wire
 		(pts
+			(xy 213.36 96.52) (xy 213.36 101.6)
+		)
+		(stroke
+			(width 0)
+			(type default)
+		)
+	)
+	(wire
+		(pts
+			(xy 218.44 91.44) (xy 218.44 101.6)
+		)
+		(stroke
+			(width 0)
+			(type default)
+		)
+	)
+	(wire
+		(pts
 			(xy 185.42 62.23) (xy 185.42 63.5)
 		)
@@
 		(pts
 			(xy 186.69 109.22) (xy 186.69 113.03)
+		)
+		(stroke
+			(width 0)
+			(type default)
+		)
+	)
+	(wire
+		(pts
+			(xy 207.01 91.44) (xy 207.01 82.55)
 		)
 		(stroke
@@
 			)
 			(justify right)
+		)
+	)
+	(symbol
+		(lib_id "Connector:Screw_Terminal_01x03")
+		(at 232.41 93.98 0)
+		(unit 1)
+		(body_style 1)
+		(exclude_from_sim no)
+		(in_bom yes)
+		(on_board yes)
+		(in_pos_files yes)
+		(dnp no)
+		(fields_autoplaced yes)
+		(property "Reference" "J3"
+			(at 234.95 93.9799 0)
+			(show_name no)
+			(do_not_autoplace no)
+			(effects
+				(font
+					(size 1.27 1.27)
+				)
+				(justify left)
+			)
+		)
+		(property "Value" "Screw_Terminal_01x03"
+			(at 234.95 95.2499 0)
+			(hide yes)
+			(show_name no)
+			(do_not_autoplace no)
+			(effects
+				(font
+					(size 1.27 1.27)
+				)
+				(justify left)
+			)
+		)
+		(property "Footprint" "TerminalBlock:TerminalBlock_Xinya_XY308-2.54-3P_1x03_P2.54mm_Horizontal"
+			(at 232.41 93.98 0)
+			(hide yes)
+			(show_name no)
+			(do_not_autoplace no)
+			(effects
+				(font
+					(size 1.27 1.27)
+				)
+			)
+		)
+		(property "Datasheet" ""
+			(at 232.41 93.98 0)
+			(hide yes)
+			(show_name no)
+			(do_not_autoplace no)
+			(effects
+				(font
+					(size 1.27 1.27)
+				)
+			)
+		)
+		(property "Description" "Generic screw terminal, single row, 01x03, script generated (kicad-library-utils/schlib/autogen/connector/)"
+			(at 232.41 93.98 0)
+			(hide yes)
+			(show_name no)
+			(do_not_autoplace no)
+			(effects
+				(font
+					(size 1.27 1.27)
+				)
+			)
+		)
+		(pin "3"
+		)
+		(pin "1"
+		)
+		(pin "2"
+		)
+		(instances
+			(project "e-foc"
+				(path "/34e5c7b2-bc7d-4136-97dd-86505a14228c/deaffcfb-90c2-4afd-9218-7765e99e9a8e"
+					(reference "J3")
+					(unit 1)
+				)
+			)
 		)
 	)
@@
 	)
 	(symbol
-		(lib_id "Connector:Screw_Terminal_01x02")
-		(at 229.87 92.71 0)
-		(unit 1)
-		(body_style 1)
-		(exclude_from_sim no)
-		(in_bom yes)
-		(on_board yes)
-		(in_pos_files yes)
-		(dnp no)
-		(fields_autoplaced yes)
-		(property "Reference" "J3"
-			(at 232.41 92.7099 0)
-			(show_name no)
-			(do_not_autoplace no)
-			(effects
-				(font
-					(size 1.27 1.27)
-				)
-				(justify left)
-			)
-		)
-		(property "Value" "Screw_Terminal_01x02"
-			(at 232.41 95.2499 0)
-			(show_name no)
-			(do_not_autoplace no)
-			(effects
-				(font
-					(size 1.27 1.27)
-				)
-				(justify left)
-			)
-		)
-		(property "Footprint" "TerminalBlock_TE-Connectivity:TerminalBlock_TE_282834-2_1x02_P2.54mm_Horizontal"
-			(at 229.87 92.71 0)
-			(hide yes)
-			(show_name no)
-			(do_not_autoplace no)
-			(effects
-				(font
-					(size 1.27 1.27)
-				)
-			)
-		)
-		(property "Datasheet" ""
-			(at 229.87 92.71 0)
-			(hide yes)
-			(show_name no)
-			(do_not_autoplace no)
-			(effects
-				(font
-					(size 1.27 1.27)
-				)
-			)
-		)
-		(property "Description" "Generic screw terminal, single row, 01x02, script generated (kicad-library-utils/schlib/autogen/connector/)"
-			(at 229.87 92.71 0)
-			(hide yes)
-			(show_name no)
-			(do_not_autoplace no)
-			(effects
-				(font
-					(size 1.27 1.27)
-				)
-			)
-		)
-		(pin "2"
-		)
-		(pin "1"
-		)
-		(instances
-			(project "e-foc"
-				(path "/34e5c7b2-bc7d-4136-97dd-86505a14228c/deaffcfb-90c2-4afd-9218-7765e99e9a8e"
-					(reference "J3")
-					(unit 1)
-				)
-			)
-		)
-	)
-	(symbol
 		(lib_id "Interface_CAN_LIN:SN65HVD230")
 		(at 173.99 92.71 0)
@@
 					(unit 1)
 				)
+			)
+		)
+	)
+	(symbol
+		(lib_id "power:GND")
+		(at 224.79 97.79 0)
+		(unit 1)
+		(body_style 1)
+		(exclude_from_sim no)
+		(in_bom yes)
+		(on_board yes)
+		(in_pos_files yes)
+		(dnp no)
+		(fields_autoplaced yes)
+		(property "Reference" "#PWR055"
+			(at 224.79 104.14 0)
+			(hide yes)
+			(show_name no)
+			(do_not_autoplace no)
+			(effects
+				(font
+					(size 1.27 1.27)
+				)
+			)
+		)
+		(property "Value" "GND"
+			(at 224.79 102.87 0)
+			(show_name no)
+			(do_not_autoplace no)
+			(effects
+				(font
+					(size 1.27 1.27)
+				)
+			)
+		)
+		(property "Footprint" ""
+			(at 224.79 97.79 0)
+			(hide yes)
+			(show_name no)
+			(do_not_autoplace no)
+			(effects
+				(font
+					(size 1.27 1.27)
+				)
+			)
+		)
+		(property "Datasheet" ""
+			(at 224.79 97.79 0)
+			(hide yes)
+			(show_name no)
+			(do_not_autoplace no)
+			(effects
+				(font
+					(size 1.27 1.27)
+				)
+			)
+		)
+		(property "Description" "Power symbol creates a global label with name \"GND\" , ground"
+			(at 224.79 97.79 0)
+			(hide yes)
+			(show_name no)
+			(do_not_autoplace no)
+			(effects
+				(font
+					(size 1.27 1.27)
+				)
+			)
+		)
+		(pin "1"
+		)
+		(instances
+			(project "e-foc"
+				(path "/34e5c7b2-bc7d-4136-97dd-86505a14228c/deaffcfb-90c2-4afd-9218-7765e99e9a8e"
+					(reference "#PWR055")
+					(unit 1)
+				)
