File: hardware/schematic/driver.kicad_sch (KiCad schematic)
At the start: 46 parts, among them Q3 CSD19506KTT, Q4 CSD19506KTT, Q5 CSD19506KTT, Q6 CSD19506KTT, Q7 CSD19506KTT, Q8 CSD19506KTT, U7 FAN7888

Commit message: refactor structure
Parts:
- gave numbers to parts that had none: 39
- renumbered Q5 to Q2, Q6 to Q3, Q3 to Q4, Q4 to Q5, Q7 to Q6, Q8 to Q7, U7 to U4
Connections:
- net GND: no longer C11.2, C12.2, C13.2, J2.1 (Pin_1), J2.2 (Pin_2), J2.3 (Pin_3), Q2.3, Q3.4, Q4.3, Q5.4, Q6.3, Q7.4, TP12.1, TP13.1, TP14.1, U4.14 (VS2), U4.18 (VS1), U4.8 (VS3)
- new net VS1: C11.2, J2.1 (Pin_1), Q2.3, Q3.4, TP14.1, U4.18 (VS1)
- new net VS2: C12.2, J2.2 (Pin_2), Q4.3, Q5.4, TP13.1, U4.14 (VS2)
- new net VS3: C13.2, J2.3 (Pin_3), Q6.3, Q7.4, TP12.1, U4.8 (VS3)

Commit message: schematic finished
Parts:
- added C15, C16: 330uF/100V, Capacitor_SMD:CP_Elec_18x22, symbol Device:C_Polarized
- renumbered C10 to C11, C11 to C12, C12 to C13, C13 to C14, D2 to D4, D3 to D5, D4 to D6, R11 to R10, R12 to R11, R13 to R12, R14 to R13, R15 to R14, R16 to R15, R17 to R16, R18 to R17, R19 to R18, R20 to R19, R21 to R20, R22 to R21, R23 to R22, R24 to R23, R25 to R24, R26 to R25, R27 to R26, R28 to R27, R29 to R28, R30 to R29, R9 to R8, R10 to R9
Connections:
- net CURRENT_B_LOW is gone; now on net CUR_A_L: R25.2, R26.1
- net GNDPWR: now also C15.2, C16.2
- net Vdrive: now also C15.1, C16.1
- net CURRENT_A_HIGH renamed CUR_A_H
- net CURRENT_A_LOW renamed CUR_A_L
- net CURRENT_B_HIGH renamed CUR_B_H
- net CURRENT_C_HIGH renamed CUR_C_H
- net PWM_A_N renamed PWM_A_L
- net PWM_B_N renamed PWM_B_L
- net PWM_C_N renamed PWM_C_L

Commit message: pcb improvements
Parts:
- removed C16: 330uF/100V, Capacitor_SMD:CP_Elec_18x22, symbol Device:C_Polarized
- removed Q2, Q3, Q4, Q5, Q6, Q7: CSD19506KTT, CSD19506KTT:TRANS_CSD19506KTT, symbol CSD19506KTT:CSD19506KTT
- added C14: 100uF/100V, Capacitor_SMD:CP_Elec_10x10.5, symbol Device:C_Polarized
- added NT2, NT3, NT4, NT5, NT6, NT7, NT8, NT9: NetTie_3_Tee, NetTie:NetTie-3_SMD_Pad0.5mm, symbol Device:NetTie_3_Tee
- added Q1, Q2, Q3: CSD88537ND, Package_SO:SOIC-8_3.9x4.9mm_P1.27mm, symbol CSD88537ND:CSD88537ND
- C10: renamed from C11; footprint (none) -> Capacitor_SMD:C_0805_2012Metric_Pad1.18x1.45mm_HandSolder
- C11: renamed from C12; footprint (none) -> Capacitor_SMD:C_1206_3216Metric_Pad1.33x1.80mm_HandSolder
- C12: renamed from C13; footprint (none) -> Capacitor_SMD:C_1206_3216Metric_Pad1.33x1.80mm_HandSolder
- C13: renamed from C14; footprint (none) -> Capacitor_SMD:C_1206_3216Metric_Pad1.33x1.80mm_HandSolder
- C15: value 330uF/100V -> 100uF/100V; footprint Capacitor_SMD:CP_Elec_18x22 -> Capacitor_SMD:CP_Elec_10x10.5
- J2: footprint TerminalBlock:TerminalBlock_Xinya_XY308-2.54-3P_1x03_P2.54mm_Horizontal -> TerminalBlock_CUI:TerminalBlock_CUI_TB007-508-03_1x03_P5.08mm_Horizontal
- renumbered D4 to D3, D5 to D4, D6 to D5, R11 to R10, R12 to R11, R13 to R12, R14 to R13, R15 to R14, R16 to R15, R17 to R16, R18 to R17, R19 to R18, R20 to R19, R21 to R20, R22 to R21, R23 to R22, R24 to R23, R25 to R24, R26 to R25, R27 to R26, R28 to R27, R29 to R28, R8 to R7, R9 to R8, R10 to R9
Connections:
- net GNDPWR: now also C14.2, NT7.1, NT7.2
- net VS1: now also Q1.1 (S), Q1.5 (D), Q1.6 (D)
- net VS2: now also Q2.1 (S), Q2.5 (D), Q2.6 (D)
- net VS3: now also Q3.1 (S), Q3.5 (D), Q3.6 (D)
- net Vdrive: now also C14.1, Q1.7 (D), Q1.8 (D), Q2.7 (D), Q2.8 (D), Q3.7 (D), Q3.8 (D)
- net at R22.1: now also Q2.2 (G)
- net at R20.1: now also Q1.4 (G)
- net at R19.1: now also Q1.2 (G)
- net at R27.1: now also Q3.4 (G)
- net at R23.1: now also Q2.4 (G)
- net at R26.1: now also Q3.2 (G)
- net CUR_A_H: no longer names the net of R21.1
- net CUR_A_H: now also NT2.1, NT2.2, Q1.3 (S)
- net CUR_A_L: no longer names the net of R21.2, R24.2, R25.1, R28.2
- net CUR_A_L: now also NT3.1, NT3.2, NT5.1, NT5.2, NT6.1, NT6.2, NT9.1, NT9.2
- net CUR_B_H: no longer names the net of R24.1
- net CUR_B_H: now also NT4.1, NT4.2, Q2.3 (S)
- net CUR_C_H: no longer names the net of R28.1
- net CUR_C_H: now also NT8.1, NT8.2, Q3.3 (S)
- new net CUR_A_N: NT3.3
- new net CUR_A_P: NT2.3
- new net CUR_B_N: NT5.3
- new net CUR_B_P: NT4.3
- new net CUR_C_N: NT9.3
- new net CUR_C_P: NT8.3
- new net CUR_TOTAL_N: NT7.3
- new net CUR_TOTAL_P: NT6.3
Other:
- moved on the sheet: C15, R19, R21, R22, R24, R25, R26, R28

Commit message: updates
Connections:
- net +20V renamed +15V
Changed lines of the file:
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@@
 			)
 		)
-		(property "Value" "+20V"
+		(property "Value" "+15V"
 			(at 102.87 46.99 0)
 			(show_name no)
@@
 			)
 		)
-		(property "Value" "+20V"
+		(property "Value" "+15V"
 			(at 102.87 134.62 0)
 			(show_name no)
@@
 			)
 		)
-		(property "Value" "+20V"
+		(property "Value" "+15V"
 			(at 102.87 73.66 0)
 			(show_name no)
