File: hardware/schematic/eeprom-mem.kicad_sch (KiCad schematic)
At the start: 10 parts

Commit message: refactor structure
Parts:
- gave numbers to parts that had none: 10
Changed lines of the file:
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@@
 		(dnp no)
 		(fields_autoplaced yes)
-		(property "Reference" "#PWR059"
+		(property "Reference" "#PWR043"
 			(at 106.68 91.44 0)
 			(hide yes)
@@
 			(project "e-foc"
 				(path "/34e5c7b2-bc7d-4136-97dd-86505a14228c/b0618b8d-c5c3-47f9-a556-34b07b48b258"
-					(reference "#PWR059")
+					(reference "#PWR043")
 					(unit 1)
 				)
@@
 		(dnp no)
 		(fields_autoplaced yes)
-		(property "Reference" "#PWR050"
+		(property "Reference" "#PWR049"
 			(at 139.7 91.44 0)
 			(hide yes)
@@
 			(project "e-foc"
 				(path "/34e5c7b2-bc7d-4136-97dd-86505a14228c/b0618b8d-c5c3-47f9-a556-34b07b48b258"
-					(reference "#PWR050")
+					(reference "#PWR049")
 					(unit 1)
 				)
@@
 		(in_pos_files yes)
 		(dnp no)
-		(property "Reference" "R?"
+		(property "Reference" "R55"
 			(at 156.21 91.4399 0)
 			(show_name no)
@@
 			(project "e-foc"
 				(path "/34e5c7b2-bc7d-4136-97dd-86505a14228c/b0618b8d-c5c3-47f9-a556-34b07b48b258"
-					(reference "R?")
+					(reference "R55")
 					(unit 1)
 				)
@@
 		(dnp no)
 		(fields_autoplaced yes)
-		(property "Reference" "#PWR057"
+		(property "Reference" "#PWR047"
 			(at 124.46 91.44 0)
 			(hide yes)
@@
 			(project "e-foc"
 				(path "/34e5c7b2-bc7d-4136-97dd-86505a14228c/b0618b8d-c5c3-47f9-a556-34b07b48b258"
-					(reference "#PWR057")
+					(reference "#PWR047")
 					(unit 1)
 				)
@@
 		(dnp no)
 		(fields_autoplaced yes)
-		(property "Reference" "#PWR061"
+		(property "Reference" "#PWR046"
 			(at 115.57 120.65 0)
 			(hide yes)
@@
 			(project "e-foc"
 				(path "/34e5c7b2-bc7d-4136-97dd-86505a14228c/b0618b8d-c5c3-47f9-a556-34b07b48b258"
-					(reference "#PWR061")
+					(reference "#PWR046")
 					(unit 1)
 				)
@@
 		(dnp no)
 		(fields_autoplaced yes)
-		(property "Reference" "#PWR052"
+		(property "Reference" "#PWR054"
 			(at 179.07 118.11 0)
 			(hide yes)
@@
 			(project "e-foc"
 				(path "/34e5c7b2-bc7d-4136-97dd-86505a14228c/b0618b8d-c5c3-47f9-a556-34b07b48b258"
-					(reference "#PWR052")
+					(reference "#PWR054")
 					(unit 1)
 				)
@@
 		(in_pos_files yes)
 		(dnp no)
-		(property "Reference" "R?"
+		(property "Reference" "R54"
 			(at 127 107.9499 0)
 			(show_name no)
@@
 			(project "e-foc"
 				(path "/34e5c7b2-bc7d-4136-97dd-86505a14228c/b0618b8d-c5c3-47f9-a556-34b07b48b258"
-					(reference "R?")
+					(reference "R54")
 					(unit 1)
 				)
@@
 		(in_pos_files yes)
 		(dnp no)
-		(property "Reference" "R?"
+		(property "Reference" "R50"
 			(at 109.22 107.9499 0)
 			(show_name no)
@@
 			(project "e-foc"
 				(path "/34e5c7b2-bc7d-4136-97dd-86505a14228c/b0618b8d-c5c3-47f9-a556-34b07b48b258"
-					(reference "R?")
+					(reference "R50")
 					(unit 1)
 				)
@@
 		(dnp no)
 		(fields_autoplaced yes)
-		(property "Reference" "#PWR060"
+		(property "Reference" "#PWR048"
 			(at 124.46 120.65 0)
 			(hide yes)
@@
 			(project "e-foc"
 				(path "/34e5c7b2-bc7d-4136-97dd-86505a14228c/b0618b8d-c5c3-47f9-a556-34b07b48b258"
-					(reference "#PWR060")
+					(reference "#PWR048")
 					(unit 1)
 				)
@@
 		(dnp no)
 		(fields_autoplaced yes)
-		(property "Reference" "#PWR062"
+		(property "Reference" "#PWR044"
 			(at 106.68 120.65 0)
 			(hide yes)
@@
 			(project "e-foc"
 				(path "/34e5c7b2-bc7d-4136-97dd-86505a14228c/b0618b8d-c5c3-47f9-a556-34b07b48b258"
-					(reference "#PWR062")
+					(reference "#PWR044")
 					(unit 1)
 				)
@@
 		(in_pos_files yes)
 		(dnp no)
-		(property "Reference" "C?"
+		(property "Reference" "C25"
 			(at 182.88 118.1099 0)
 			(show_name no)
@@
 			(project "e-foc"
 				(path "/34e5c7b2-bc7d-4136-97dd-86505a14228c/b0618b8d-c5c3-47f9-a556-34b07b48b258"
-					(reference "C?")
+					(reference "C25")
 					(unit 1)
 				)
@@
 		(dnp no)
 		(fields_autoplaced yes)
-		(property "Reference" "#PWR054"
+		(property "Reference" "#PWR051"
 			(at 152.4 120.65 0)
 			(hide yes)
@@
 			(project "e-foc"
 				(path "/34e5c7b2-bc7d-4136-97dd-86505a14228c/b0618b8d-c5c3-47f9-a556-34b07b48b258"
-					(reference "#PWR054")
+					(reference "#PWR051")
 					(unit 1)
 				)
@@
 		(dnp no)
 		(fields_autoplaced yes)
-		(property "Reference" "U?"
+		(property "Reference" "U8"
 			(at 141.8433 91.44 0)
 			(show_name no)
@@
 			(project "e-foc"
 				(path "/34e5c7b2-bc7d-4136-97dd-86505a14228c/b0618b8d-c5c3-47f9-a556-34b07b48b258"
-					(reference "U?")
+					(reference "U8")
 					(unit 1)
 				)
@@
 		(dnp no)
 		(fields_autoplaced yes)
-		(property "Reference" "#PWR058"
+		(property "Reference" "#PWR045"
 			(at 115.57 91.44 0)
 			(hide yes)
@@
 			(project "e-foc"
 				(path "/34e5c7b2-bc7d-4136-97dd-86505a14228c/b0618b8d-c5c3-47f9-a556-34b07b48b258"
-					(reference "#PWR058")
+					(reference "#PWR045")
 					(unit 1)
 				)
@@
 		(in_pos_files yes)
 		(dnp no)
-		(property "Reference" "R?"
+		(property "Reference" "R56"
 			(at 166.37 91.4399 0)
 			(show_name no)
@@
 			(project "e-foc"
 				(path "/34e5c7b2-bc7d-4136-97dd-86505a14228c/b0618b8d-c5c3-47f9-a556-34b07b48b258"
-					(reference "R?")
+					(reference "R56")
 					(unit 1)
 				)
@@
 		(in_pos_files yes)
 		(dnp no)
-		(property "Reference" "R?"
+		(property "Reference" "R52"
 			(at 118.11 107.9499 0)
 			(show_name no)
@@
 			(project "e-foc"
 				(path "/34e5c7b2-bc7d-4136-97dd-86505a14228c/b0618b8d-c5c3-47f9-a556-34b07b48b258"
-					(reference "R?")
+					(reference "R52")
 					(unit 1)
 				)
@@
 		(dnp no)
 		(fields_autoplaced yes)
-		(property "Reference" "#PWR051"
+		(property "Reference" "#PWR050"
 			(at 139.7 120.65 0)
 			(hide yes)
@@
 			(project "e-foc"
 				(path "/34e5c7b2-bc7d-4136-97dd-86505a14228c/b0618b8d-c5c3-47f9-a556-34b07b48b258"
-					(reference "#PWR051")
+					(reference "#PWR050")
 					(unit 1)
 				)
@@
 		(dnp no)
 		(fields_autoplaced yes)
-		(property "Reference" "#PWR056"
+		(property "Reference" "#PWR053"
 			(at 163.83 91.44 0)
 			(hide yes)
@@
 			(project "e-foc"
 				(path "/34e5c7b2-bc7d-4136-97dd-86505a14228c/b0618b8d-c5c3-47f9-a556-34b07b48b258"
-					(reference "#PWR056")
+					(reference "#PWR053")
 					(unit 1)
 				)
@@
 		(dnp no)
 		(fields_autoplaced yes)
-		(property "Reference" "#PWR055"
+		(property "Reference" "#PWR052"
 			(at 153.67 91.44 0)
 			(hide yes)
@@
 			(project "e-foc"
 				(path "/34e5c7b2-bc7d-4136-97dd-86505a14228c/b0618b8d-c5c3-47f9-a556-34b07b48b258"
-					(reference "#PWR055")
+					(reference "#PWR052")
 					(unit 1)
 				)
@@
 		(in_pos_files yes)
 		(dnp yes)
-		(property "Reference" "R?"
+		(property "Reference" "R53"
 			(at 127 91.4399 0)
 			(show_name no)
@@
 			(project "e-foc"
 				(path "/34e5c7b2-bc7d-4136-97dd-86505a14228c/b0618b8d-c5c3-47f9-a556-34b07b48b258"
-					(reference "R?")
+					(reference "R53")
 					(unit 1)
 				)
@@
 		(in_pos_files yes)
 		(dnp yes)
-		(property "Reference" "R?"
+		(property "Reference" "R49"
 			(at 109.22 91.4399 0)
 			(show_name no)
@@
 			(project "e-foc"
 				(path "/34e5c7b2-bc7d-4136-97dd-86505a14228c/b0618b8d-c5c3-47f9-a556-34b07b48b258"
-					(reference "R?")
+					(reference "R49")
 					(unit 1)
 				)
@@
 		(dnp no)
 		(fields_autoplaced yes)
-		(property "Reference" "#PWR053"
+		(property "Reference" "#PWR055"
 			(at 179.07 130.81 0)
 			(hide yes)
@@
 			(project "e-foc"
 				(path "/34e5c7b2-bc7d-4136-97dd-86505a14228c/b0618b8d-c5c3-47f9-a556-34b07b48b258"
-					(reference "#PWR053")
+					(reference "#PWR055")
 					(unit 1)
 				)
@@
 		(in_pos_files yes)
 		(dnp yes)
-		(property "Reference" "R?"
+		(property "Reference" "R51"
 			(at 118.11 91.4399 0)
 			(show_name no)
@@
 			(project "e-foc"
 				(path "/34e5c7b2-bc7d-4136-97dd-86505a14228c/b0618b8d-c5c3-47f9-a556-34b07b48b258"
-					(reference "R?")
-					(unit 1)
-				)
+					(reference "R51")
+					(unit 1)
+				)

Commit message: schematic finished
Parts:
- renumbered C25 to C32, R49 to R53, R50 to R54, R51 to R55, R52 to R56, R53 to R57, R54 to R58, R55 to R59, R56 to R60
Changed lines of the file:
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@@
 		)
 	)
-	(global_label "I2C_SDA"
-		(shape input)
-		(at 166.37 99.06 0)
-		(fields_autoplaced yes)
+	(hierarchical_label "I2C_SCL"
+		(shape output)
+		(at 166.37 101.6 0)
 		(effects
 			(font
@@
 			(justify left)
 		)
-		(property "Intersheetrefs" "${INTERSHEET_REFS}"
-			(at 176.9752 99.06 0)
-			(hide yes)
-			(show_name no)
-			(do_not_autoplace no)
-			(effects
-				(font
-					(size 1.27 1.27)
-				)
-				(justify left)
-			)
-		)
-	)
-	(global_label "I2C_SCL"
-		(shape input)
-		(at 166.37 101.6 0)
-		(fields_autoplaced yes)
+	)
+	(hierarchical_label "I2C_SDA"
+		(shape output)
+		(at 166.37 99.06 0)
 		(effects
 			(font
@@
 			(justify left)
 		)
-		(property "Intersheetrefs" "${INTERSHEET_REFS}"
-			(at 176.9147 101.6 0)
-			(hide yes)
-			(show_name no)
-			(do_not_autoplace no)
-			(effects
-				(font
-					(size 1.27 1.27)
-				)
-				(justify left)
-			)
-		)
 	)
 	(symbol
@@
 		(dnp no)
 		(fields_autoplaced yes)
-		(property "Reference" "#PWR043"
+		(property "Reference" "#PWR057"
 			(at 106.68 91.44 0)
 			(hide yes)
@@
 			(project "e-foc"
 				(path "/34e5c7b2-bc7d-4136-97dd-86505a14228c/b0618b8d-c5c3-47f9-a556-34b07b48b258"
-					(reference "#PWR043")
+					(reference "#PWR057")
 					(unit 1)
 				)
@@
 		(dnp no)
 		(fields_autoplaced yes)
-		(property "Reference" "#PWR049"
+		(property "Reference" "#PWR063"
 			(at 139.7 91.44 0)
 			(hide yes)
@@
 			(project "e-foc"
 				(path "/34e5c7b2-bc7d-4136-97dd-86505a14228c/b0618b8d-c5c3-47f9-a556-34b07b48b258"
-					(reference "#PWR049")
+					(reference "#PWR063")
 					(unit 1)
 				)
@@
 		(in_pos_files yes)
 		(dnp no)
-		(property "Reference" "R55"
+		(property "Reference" "R59"
 			(at 156.21 91.4399 0)
 			(show_name no)
@@
 			(project "e-foc"
 				(path "/34e5c7b2-bc7d-4136-97dd-86505a14228c/b0618b8d-c5c3-47f9-a556-34b07b48b258"
-					(reference "R55")
+					(reference "R59")
 					(unit 1)
 				)
@@
 		(dnp no)
 		(fields_autoplaced yes)
-		(property "Reference" "#PWR047"
+		(property "Reference" "#PWR061"
 			(at 124.46 91.44 0)
 			(hide yes)
@@
 			(project "e-foc"
 				(path "/34e5c7b2-bc7d-4136-97dd-86505a14228c/b0618b8d-c5c3-47f9-a556-34b07b48b258"
-					(reference "#PWR047")
+					(reference "#PWR061")
 					(unit 1)
 				)
@@
 		(dnp no)
 		(fields_autoplaced yes)
-		(property "Reference" "#PWR046"
+		(property "Reference" "#PWR060"
 			(at 115.57 120.65 0)
 			(hide yes)
@@
 			(project "e-foc"
 				(path "/34e5c7b2-bc7d-4136-97dd-86505a14228c/b0618b8d-c5c3-47f9-a556-34b07b48b258"
-					(reference "#PWR046")
+					(reference "#PWR060")
 					(unit 1)
 				)
@@
 		(dnp no)
 		(fields_autoplaced yes)
-		(property "Reference" "#PWR054"
+		(property "Reference" "#PWR068"
 			(at 179.07 118.11 0)
 			(hide yes)
@@
 			(project "e-foc"
 				(path "/34e5c7b2-bc7d-4136-97dd-86505a14228c/b0618b8d-c5c3-47f9-a556-34b07b48b258"
-					(reference "#PWR054")
+					(reference "#PWR068")
 					(unit 1)
 				)
@@
 		(in_pos_files yes)
 		(dnp no)
-		(property "Reference" "R54"
+		(property "Reference" "R58"
 			(at 127 107.9499 0)
 			(show_name no)
@@
 			(project "e-foc"
 				(path "/34e5c7b2-bc7d-4136-97dd-86505a14228c/b0618b8d-c5c3-47f9-a556-34b07b48b258"
-					(reference "R54")
+					(reference "R58")
 					(unit 1)
 				)
@@
 		(in_pos_files yes)
 		(dnp no)
-		(property "Reference" "R50"
+		(property "Reference" "R54"
 			(at 109.22 107.9499 0)
 			(show_name no)
@@
 			(project "e-foc"
 				(path "/34e5c7b2-bc7d-4136-97dd-86505a14228c/b0618b8d-c5c3-47f9-a556-34b07b48b258"
-					(reference "R50")
+					(reference "R54")
 					(unit 1)
 				)
@@
 		(dnp no)
 		(fields_autoplaced yes)
-		(property "Reference" "#PWR048"
+		(property "Reference" "#PWR062"
 			(at 124.46 120.65 0)
 			(hide yes)
@@
 			(project "e-foc"
 				(path "/34e5c7b2-bc7d-4136-97dd-86505a14228c/b0618b8d-c5c3-47f9-a556-34b07b48b258"
-					(reference "#PWR048")
+					(reference "#PWR062")
 					(unit 1)
 				)
@@
 		(dnp no)
 		(fields_autoplaced yes)
-		(property "Reference" "#PWR044"
+		(property "Reference" "#PWR058"
 			(at 106.68 120.65 0)
 			(hide yes)
@@
 			(project "e-foc"
 				(path "/34e5c7b2-bc7d-4136-97dd-86505a14228c/b0618b8d-c5c3-47f9-a556-34b07b48b258"
-					(reference "#PWR044")
+					(reference "#PWR058")
 					(unit 1)
 				)
@@
 		(in_pos_files yes)
 		(dnp no)
-		(property "Reference" "C25"
+		(property "Reference" "C32"
 			(at 182.88 118.1099 0)
 			(show_name no)
@@
 			(project "e-foc"
 				(path "/34e5c7b2-bc7d-4136-97dd-86505a14228c/b0618b8d-c5c3-47f9-a556-34b07b48b258"
-					(reference "C25")
+					(reference "C32")
 					(unit 1)
 				)
@@
 		(dnp no)
 		(fields_autoplaced yes)
-		(property "Reference" "#PWR051"
+		(property "Reference" "#PWR065"
 			(at 152.4 120.65 0)
 			(hide yes)
@@
 			(project "e-foc"
 				(path "/34e5c7b2-bc7d-4136-97dd-86505a14228c/b0618b8d-c5c3-47f9-a556-34b07b48b258"
-					(reference "#PWR051")
+					(reference "#PWR065")
 					(unit 1)
 				)
@@
 		(dnp no)
 		(fields_autoplaced yes)
-		(property "Reference" "#PWR045"
+		(property "Reference" "#PWR059"
 			(at 115.57 91.44 0)
 			(hide yes)
@@
 			(project "e-foc"
 				(path "/34e5c7b2-bc7d-4136-97dd-86505a14228c/b0618b8d-c5c3-47f9-a556-34b07b48b258"
-					(reference "#PWR045")
+					(reference "#PWR059")
 					(unit 1)
 				)
@@
 		(in_pos_files yes)
 		(dnp no)
-		(property "Reference" "R56"
+		(property "Reference" "R60"
 			(at 166.37 91.4399 0)
 			(show_name no)
@@
 			(project "e-foc"
 				(path "/34e5c7b2-bc7d-4136-97dd-86505a14228c/b0618b8d-c5c3-47f9-a556-34b07b48b258"
-					(reference "R56")
+					(reference "R60")
 					(unit 1)
 				)
@@
 		(in_pos_files yes)
 		(dnp no)
-		(property "Reference" "R52"
+		(property "Reference" "R56"
 			(at 118.11 107.9499 0)
 			(show_name no)
@@
 			(project "e-foc"
 				(path "/34e5c7b2-bc7d-4136-97dd-86505a14228c/b0618b8d-c5c3-47f9-a556-34b07b48b258"
-					(reference "R52")
+					(reference "R56")
 					(unit 1)
 				)
@@
 		(dnp no)
 		(fields_autoplaced yes)
-		(property "Reference" "#PWR050"
+		(property "Reference" "#PWR064"
 			(at 139.7 120.65 0)
 			(hide yes)
@@
 			(project "e-foc"
 				(path "/34e5c7b2-bc7d-4136-97dd-86505a14228c/b0618b8d-c5c3-47f9-a556-34b07b48b258"
-					(reference "#PWR050")
+					(reference "#PWR064")
 					(unit 1)
 				)
@@
 		(dnp no)
 		(fields_autoplaced yes)
-		(property "Reference" "#PWR053"
+		(property "Reference" "#PWR067"
 			(at 163.83 91.44 0)
 			(hide yes)
@@
 			(project "e-foc"
 				(path "/34e5c7b2-bc7d-4136-97dd-86505a14228c/b0618b8d-c5c3-47f9-a556-34b07b48b258"
-					(reference "#PWR053")
+					(reference "#PWR067")
 					(unit 1)
 				)
@@
 		(dnp no)
 		(fields_autoplaced yes)
-		(property "Reference" "#PWR052"
+		(property "Reference" "#PWR066"
 			(at 153.67 91.44 0)
 			(hide yes)
@@
 			(project "e-foc"
 				(path "/34e5c7b2-bc7d-4136-97dd-86505a14228c/b0618b8d-c5c3-47f9-a556-34b07b48b258"
-					(reference "#PWR052")
+					(reference "#PWR066")
 					(unit 1)
 				)
@@
 		(in_pos_files yes)
 		(dnp yes)
-		(property "Reference" "R53"
+		(property "Reference" "R57"
 			(at 127 91.4399 0)
 			(show_name no)
@@
 			(project "e-foc"
 				(path "/34e5c7b2-bc7d-4136-97dd-86505a14228c/b0618b8d-c5c3-47f9-a556-34b07b48b258"
-					(reference "R53")
+					(reference "R57")
 					(unit 1)
 				)
@@
 		(in_pos_files yes)
 		(dnp yes)
-		(property "Reference" "R49"
+		(property "Reference" "R53"
 			(at 109.22 91.4399 0)
 			(show_name no)
@@
 			(project "e-foc"
 				(path "/34e5c7b2-bc7d-4136-97dd-86505a14228c/b0618b8d-c5c3-47f9-a556-34b07b48b258"
-					(reference "R49")
+					(reference "R53")
 					(unit 1)
 				)
@@
 		(dnp no)
 		(fields_autoplaced yes)
-		(property "Reference" "#PWR055"
+		(property "Reference" "#PWR069"
 			(at 179.07 130.81 0)
 			(hide yes)
@@
 			(project "e-foc"
 				(path "/34e5c7b2-bc7d-4136-97dd-86505a14228c/b0618b8d-c5c3-47f9-a556-34b07b48b258"
-					(reference "#PWR055")
+					(reference "#PWR069")
 					(unit 1)
 				)
@@
 		(in_pos_files yes)
 		(dnp yes)
-		(property "Reference" "R51"
+		(property "Reference" "R55"
 			(at 118.11 91.4399 0)
 			(show_name no)
@@
 			(project "e-foc"
 				(path "/34e5c7b2-bc7d-4136-97dd-86505a14228c/b0618b8d-c5c3-47f9-a556-34b07b48b258"
-					(reference "R51")
-					(unit 1)
-				)
+					(reference "R55")
+					(unit 1)
+				)
