File: hardware/schematic/flash-mem.kicad_sch (KiCad schematic)
At the start: 6 parts, among them U2 W25Q32JVSS

Commit message: refactor structure
Parts:
- gave numbers to parts that had none: 5
- renumbered U2 to U9
Changed lines of the file:
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@@
 		(in_pos_files yes)
 		(dnp no)
-		(property "Reference" "R?"
+		(property "Reference" "R59"
 			(at 124.968 95.25 90)
 			(show_name no)
@@
 			(project "e-foc"
 				(path "/34e5c7b2-bc7d-4136-97dd-86505a14228c/6cd2b0a0-683f-4196-92a9-4a51f926d77e"
-					(reference "R?")
+					(reference "R59")
 					(unit 1)
 				)
@@
 		(dnp no)
 		(fields_autoplaced yes)
-		(property "Reference" "#PWR045"
+		(property "Reference" "#PWR059"
 			(at 146.05 105.41 0)
 			(hide yes)
@@
 			(project "e-foc"
 				(path "/34e5c7b2-bc7d-4136-97dd-86505a14228c/6cd2b0a0-683f-4196-92a9-4a51f926d77e"
-					(reference "#PWR045")
+					(reference "#PWR059")
 					(unit 1)
 				)
@@
 		(in_pos_files yes)
 		(dnp no)
-		(property "Reference" "R?"
+		(property "Reference" "R60"
 			(at 135.89 71.1199 0)
 			(show_name no)
@@
 			(project "e-foc"
 				(path "/34e5c7b2-bc7d-4136-97dd-86505a14228c/6cd2b0a0-683f-4196-92a9-4a51f926d77e"
-					(reference "R?")
+					(reference "R60")
 					(unit 1)
 				)
@@
 		(dnp no)
 		(fields_autoplaced yes)
-		(property "Reference" "#PWR049"
+		(property "Reference" "#PWR060"
 			(at 175.26 83.82 0)
 			(hide yes)
@@
 			(project "e-foc"
 				(path "/34e5c7b2-bc7d-4136-97dd-86505a14228c/6cd2b0a0-683f-4196-92a9-4a51f926d77e"
-					(reference "#PWR049")
+					(reference "#PWR060")
 					(unit 1)
 				)
@@
 		(dnp no)
 		(fields_autoplaced yes)
-		(property "Reference" "#PWR046"
+		(property "Reference" "#PWR057"
 			(at 133.35 69.85 0)
 			(hide yes)
@@
 			(project "e-foc"
 				(path "/34e5c7b2-bc7d-4136-97dd-86505a14228c/6cd2b0a0-683f-4196-92a9-4a51f926d77e"
-					(reference "#PWR046")
+					(reference "#PWR057")
 					(unit 1)
 				)
@@
 		(in_pos_files yes)
 		(dnp no)
-		(property "Reference" "R?"
+		(property "Reference" "R58"
 			(at 124.968 90.17 90)
 			(show_name no)
@@
 			(project "e-foc"
 				(path "/34e5c7b2-bc7d-4136-97dd-86505a14228c/6cd2b0a0-683f-4196-92a9-4a51f926d77e"
-					(reference "R?")
+					(reference "R58")
 					(unit 1)
 				)
@@
 		(in_pos_files yes)
 		(dnp no)
-		(property "Reference" "C?"
+		(property "Reference" "C26"
 			(at 179.07 83.8199 0)
 			(show_name no)
@@
 			(project "e-foc"
 				(path "/34e5c7b2-bc7d-4136-97dd-86505a14228c/6cd2b0a0-683f-4196-92a9-4a51f926d77e"
-					(reference "C?")
+					(reference "C26")
 					(unit 1)
 				)
@@
 		(dnp no)
 		(fields_autoplaced yes)
-		(property "Reference" "#PWR047"
+		(property "Reference" "#PWR056"
 			(at 104.14 88.9 0)
 			(hide yes)
@@
 			(project "e-foc"
 				(path "/34e5c7b2-bc7d-4136-97dd-86505a14228c/6cd2b0a0-683f-4196-92a9-4a51f926d77e"
-					(reference "#PWR047")
+					(reference "#PWR056")
 					(unit 1)
 				)
@@
 		(dnp no)
 		(fields_autoplaced yes)
-		(property "Reference" "U2"
+		(property "Reference" "U9"
 			(at 157.48 83.8199 0)
 			(show_name no)
@@
 			(project "e-foc"
 				(path "/34e5c7b2-bc7d-4136-97dd-86505a14228c/6cd2b0a0-683f-4196-92a9-4a51f926d77e"
-					(reference "U2")
+					(reference "U9")
 					(unit 1)
 				)
@@
 		(in_pos_files yes)
 		(dnp no)
-		(property "Reference" "R?"
+		(property "Reference" "R57"
 			(at 122.936 75.692 90)
 			(show_name no)
@@
 			(project "e-foc"
 				(path "/34e5c7b2-bc7d-4136-97dd-86505a14228c/6cd2b0a0-683f-4196-92a9-4a51f926d77e"
-					(reference "R?")
+					(reference "R57")
 					(unit 1)
 				)
@@
 		(dnp no)
 		(fields_autoplaced yes)
-		(property "Reference" "#PWR048"
+		(property "Reference" "#PWR061"
 			(at 175.26 96.52 0)
 			(hide yes)
@@
 			(project "e-foc"
 				(path "/34e5c7b2-bc7d-4136-97dd-86505a14228c/6cd2b0a0-683f-4196-92a9-4a51f926d77e"
-					(reference "#PWR048")
+					(reference "#PWR061")
 					(unit 1)
 				)
@@
 		(dnp no)
 		(fields_autoplaced yes)
-		(property "Reference" "#PWR044"
+		(property "Reference" "#PWR058"
 			(at 146.05 73.66 0)
 			(hide yes)
@@
 			(project "e-foc"
 				(path "/34e5c7b2-bc7d-4136-97dd-86505a14228c/6cd2b0a0-683f-4196-92a9-4a51f926d77e"
-					(reference "#PWR044")
-					(unit 1)
-				)
+					(reference "#PWR058")
+					(unit 1)
+				)

Commit message: schematic finished
Parts:
- renumbered C26 to C33, R57 to R61, R58 to R62, R59 to R63, R60 to R64
Changed lines of the file:
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@@
 		)
 	)
-	(global_label "SPI_MISO"
-		(shape input)
+	(hierarchical_label "SPI_MISO"
+		(shape output)
 		(at 118.11 82.55 180)
-		(fields_autoplaced yes)
 		(effects
 			(font
@@
 			(justify right)
 		)
-		(property "Intersheetrefs" "${INTERSHEET_REFS}"
-			(at 106.4767 82.55 0)
-			(hide yes)
-			(show_name no)
-			(do_not_autoplace no)
-			(effects
-				(font
-					(size 1.27 1.27)
-				)
-				(justify right)
-			)
-		)
-	)
-	(global_label "SPI_CS"
-		(shape input)
-		(at 118.11 77.47 180)
-		(fields_autoplaced yes)
+	)
+	(hierarchical_label "SPI_MOSI"
+		(shape output)
+		(at 118.11 85.09 180)
 		(effects
 			(font
@@
 			(justify right)
 		)
-		(property "Intersheetrefs" "${INTERSHEET_REFS}"
-			(at 108.5934 77.47 0)
-			(hide yes)
-			(show_name no)
-			(do_not_autoplace no)
-			(effects
-				(font
-					(size 1.27 1.27)
-				)
-				(justify right)
-			)
-		)
-	)
-	(global_label "SPI_SCK"
-		(shape input)
-		(at 118.11 80.01 180)
-		(fields_autoplaced yes)
+	)
+	(hierarchical_label "SPI_CS"
+		(shape output)
+		(at 118.11 77.47 180)
 		(effects
 			(font
@@
 			(justify right)
 		)
-		(property "Intersheetrefs" "${INTERSHEET_REFS}"
-			(at 107.3234 80.01 0)
-			(hide yes)
-			(show_name no)
-			(do_not_autoplace no)
-			(effects
-				(font
-					(size 1.27 1.27)
-				)
-				(justify right)
-			)
-		)
-	)
-	(global_label "SPI_MOSI"
-		(shape input)
-		(at 118.11 85.09 180)
-		(fields_autoplaced yes)
+	)
+	(hierarchical_label "SPI_SCK"
+		(shape output)
+		(at 118.11 80.01 180)
 		(effects
 			(font
@@
 			(justify right)
 		)
-		(property "Intersheetrefs" "${INTERSHEET_REFS}"
-			(at 106.4767 85.09 0)
-			(hide yes)
-			(show_name no)
-			(do_not_autoplace no)
-			(effects
-				(font
-					(size 1.27 1.27)
-				)
-				(justify right)
-			)
-		)
 	)
 	(symbol
@@
 		(in_pos_files yes)
 		(dnp no)
-		(property "Reference" "R59"
+		(property "Reference" "R63"
 			(at 124.968 95.25 90)
 			(show_name no)
@@
 			(project "e-foc"
 				(path "/34e5c7b2-bc7d-4136-97dd-86505a14228c/6cd2b0a0-683f-4196-92a9-4a51f926d77e"
-					(reference "R59")
+					(reference "R63")
 					(unit 1)
 				)
@@
 		(dnp no)
 		(fields_autoplaced yes)
-		(property "Reference" "#PWR059"
+		(property "Reference" "#PWR073"
 			(at 146.05 105.41 0)
 			(hide yes)
@@
 			(project "e-foc"
 				(path "/34e5c7b2-bc7d-4136-97dd-86505a14228c/6cd2b0a0-683f-4196-92a9-4a51f926d77e"
-					(reference "#PWR059")
+					(reference "#PWR073")
 					(unit 1)
 				)
@@
 		(in_pos_files yes)
 		(dnp no)
-		(property "Reference" "R60"
+		(property "Reference" "R64"
 			(at 135.89 71.1199 0)
 			(show_name no)
@@
 			(project "e-foc"
 				(path "/34e5c7b2-bc7d-4136-97dd-86505a14228c/6cd2b0a0-683f-4196-92a9-4a51f926d77e"
-					(reference "R60")
+					(reference "R64")
 					(unit 1)
 				)
@@
 		(dnp no)
 		(fields_autoplaced yes)
-		(property "Reference" "#PWR060"
+		(property "Reference" "#PWR074"
 			(at 175.26 83.82 0)
 			(hide yes)
@@
 			(project "e-foc"
 				(path "/34e5c7b2-bc7d-4136-97dd-86505a14228c/6cd2b0a0-683f-4196-92a9-4a51f926d77e"
-					(reference "#PWR060")
+					(reference "#PWR074")
 					(unit 1)
 				)
@@
 		(dnp no)
 		(fields_autoplaced yes)
-		(property "Reference" "#PWR057"
+		(property "Reference" "#PWR071"
 			(at 133.35 69.85 0)
 			(hide yes)
@@
 			(project "e-foc"
 				(path "/34e5c7b2-bc7d-4136-97dd-86505a14228c/6cd2b0a0-683f-4196-92a9-4a51f926d77e"
-					(reference "#PWR057")
+					(reference "#PWR071")
 					(unit 1)
 				)
@@
 		(in_pos_files yes)
 		(dnp no)
-		(property "Reference" "R58"
+		(property "Reference" "R62"
 			(at 124.968 90.17 90)
 			(show_name no)
@@
 			(project "e-foc"
 				(path "/34e5c7b2-bc7d-4136-97dd-86505a14228c/6cd2b0a0-683f-4196-92a9-4a51f926d77e"
-					(reference "R58")
+					(reference "R62")
 					(unit 1)
 				)
@@
 		(in_pos_files yes)
 		(dnp no)
-		(property "Reference" "C26"
+		(property "Reference" "C33"
 			(at 179.07 83.8199 0)
 			(show_name no)
@@
 			(project "e-foc"
 				(path "/34e5c7b2-bc7d-4136-97dd-86505a14228c/6cd2b0a0-683f-4196-92a9-4a51f926d77e"
-					(reference "C26")
+					(reference "C33")
 					(unit 1)
 				)
@@
 		(dnp no)
 		(fields_autoplaced yes)
-		(property "Reference" "#PWR056"
+		(property "Reference" "#PWR070"
 			(at 104.14 88.9 0)
 			(hide yes)
@@
 			(project "e-foc"
 				(path "/34e5c7b2-bc7d-4136-97dd-86505a14228c/6cd2b0a0-683f-4196-92a9-4a51f926d77e"
-					(reference "#PWR056")
+					(reference "#PWR070")
 					(unit 1)
 				)
@@
 		(in_pos_files yes)
 		(dnp no)
-		(property "Reference" "R57"
+		(property "Reference" "R61"
 			(at 122.936 75.692 90)
 			(show_name no)
@@
 			(project "e-foc"
 				(path "/34e5c7b2-bc7d-4136-97dd-86505a14228c/6cd2b0a0-683f-4196-92a9-4a51f926d77e"
-					(reference "R57")
+					(reference "R61")
 					(unit 1)
 				)
@@
 		(dnp no)
 		(fields_autoplaced yes)
-		(property "Reference" "#PWR061"
+		(property "Reference" "#PWR075"
 			(at 175.26 96.52 0)
 			(hide yes)
@@
 			(project "e-foc"
 				(path "/34e5c7b2-bc7d-4136-97dd-86505a14228c/6cd2b0a0-683f-4196-92a9-4a51f926d77e"
-					(reference "#PWR061")
+					(reference "#PWR075")
 					(unit 1)
 				)
@@
 		(dnp no)
 		(fields_autoplaced yes)
-		(property "Reference" "#PWR058"
+		(property "Reference" "#PWR072"
 			(at 146.05 73.66 0)
 			(hide yes)
@@
 			(project "e-foc"
 				(path "/34e5c7b2-bc7d-4136-97dd-86505a14228c/6cd2b0a0-683f-4196-92a9-4a51f926d77e"
-					(reference "#PWR058")
-					(unit 1)
-				)
+					(reference "#PWR072")
+					(unit 1)
+				)

Commit message: pcb improvements
Parts:
- C36: renamed from C33; footprint (none) -> Capacitor_SMD:C_0805_2012Metric_Pad1.18x1.45mm_HandSolder
- renumbered R61 to R69, R62 to R70, R63 to R71, R64 to R72, U9 to U10
Changed lines of the file:
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@@
 		(in_pos_files yes)
 		(dnp no)
-		(property "Reference" "R63"
-			(at 124.968 95.25 90)
+		(property "Reference" "R71"
+			(at 123.698 94.996 90)
 			(show_name no)
 			(do_not_autoplace no)
@@
 			(project "e-foc"
 				(path "/34e5c7b2-bc7d-4136-97dd-86505a14228c/6cd2b0a0-683f-4196-92a9-4a51f926d77e"
-					(reference "R63")
+					(reference "R71")
 					(unit 1)
 				)
@@
 		(dnp no)
 		(fields_autoplaced yes)
-		(property "Reference" "#PWR073"
+		(property "Reference" "#PWR083"
 			(at 146.05 105.41 0)
 			(hide yes)
@@
 			(project "e-foc"
 				(path "/34e5c7b2-bc7d-4136-97dd-86505a14228c/6cd2b0a0-683f-4196-92a9-4a51f926d77e"
-					(reference "#PWR073")
+					(reference "#PWR083")
 					(unit 1)
 				)
@@
 		(in_pos_files yes)
 		(dnp no)
-		(property "Reference" "R64"
+		(property "Reference" "R72"
 			(at 135.89 71.1199 0)
 			(show_name no)
@@
 			(project "e-foc"
 				(path "/34e5c7b2-bc7d-4136-97dd-86505a14228c/6cd2b0a0-683f-4196-92a9-4a51f926d77e"
-					(reference "R64")
+					(reference "R72")
 					(unit 1)
 				)
@@
 		(dnp no)
 		(fields_autoplaced yes)
-		(property "Reference" "#PWR074"
+		(property "Reference" "#PWR084"
 			(at 175.26 83.82 0)
 			(hide yes)
@@
 			(project "e-foc"
 				(path "/34e5c7b2-bc7d-4136-97dd-86505a14228c/6cd2b0a0-683f-4196-92a9-4a51f926d77e"
-					(reference "#PWR074")
+					(reference "#PWR084")
 					(unit 1)
 				)
@@
 		(dnp no)
 		(fields_autoplaced yes)
-		(property "Reference" "#PWR071"
+		(property "Reference" "#PWR081"
 			(at 133.35 69.85 0)
 			(hide yes)
@@
 			(project "e-foc"
 				(path "/34e5c7b2-bc7d-4136-97dd-86505a14228c/6cd2b0a0-683f-4196-92a9-4a51f926d77e"
-					(reference "#PWR071")
+					(reference "#PWR081")
 					(unit 1)
 				)
@@
 		(in_pos_files yes)
 		(dnp no)
-		(property "Reference" "R62"
-			(at 124.968 90.17 90)
+		(property "Reference" "R70"
+			(at 123.444 90.17 90)
 			(show_name no)
 			(do_not_autoplace no)
@@
 			(project "e-foc"
 				(path "/34e5c7b2-bc7d-4136-97dd-86505a14228c/6cd2b0a0-683f-4196-92a9-4a51f926d77e"
-					(reference "R62")
+					(reference "R70")
 					(unit 1)
 				)
@@
 		(in_pos_files yes)
 		(dnp no)
-		(property "Reference" "C33"
+		(property "Reference" "C36"
 			(at 179.07 83.8199 0)
 			(show_name no)
@@
 			)
 		)
-		(property "Footprint" ""
+		(property "Footprint" "Capacitor_SMD:C_0805_2012Metric_Pad1.18x1.45mm_HandSolder"
 			(at 176.2252 88.9 0)
 			(hide yes)
@@
 			(project "e-foc"
 				(path "/34e5c7b2-bc7d-4136-97dd-86505a14228c/6cd2b0a0-683f-4196-92a9-4a51f926d77e"
-					(reference "C33")
+					(reference "C36")
 					(unit 1)
 				)
@@
 		(dnp no)
 		(fields_autoplaced yes)
-		(property "Reference" "#PWR070"
+		(property "Reference" "#PWR080"
 			(at 104.14 88.9 0)
 			(hide yes)
@@
 			(project "e-foc"
 				(path "/34e5c7b2-bc7d-4136-97dd-86505a14228c/6cd2b0a0-683f-4196-92a9-4a51f926d77e"
-					(reference "#PWR070")
+					(reference "#PWR080")
 					(unit 1)
 				)
@@
 		(dnp no)
 		(fields_autoplaced yes)
-		(property "Reference" "U9"
+		(property "Reference" "U10"
 			(at 157.48 83.8199 0)
 			(show_name no)
@@
 			(project "e-foc"
 				(path "/34e5c7b2-bc7d-4136-97dd-86505a14228c/6cd2b0a0-683f-4196-92a9-4a51f926d77e"
-					(reference "U9")
+					(reference "U10")
 					(unit 1)
 				)
@@
 		(in_pos_files yes)
 		(dnp no)
-		(property "Reference" "R61"
-			(at 122.936 75.692 90)
+		(property "Reference" "R69"
+			(at 121.92 75.692 90)
 			(show_name no)
 			(do_not_autoplace no)
@@
 			(project "e-foc"
 				(path "/34e5c7b2-bc7d-4136-97dd-86505a14228c/6cd2b0a0-683f-4196-92a9-4a51f926d77e"
-					(reference "R61")
+					(reference "R69")
 					(unit 1)
 				)
@@
 		(dnp no)
 		(fields_autoplaced yes)
-		(property "Reference" "#PWR075"
+		(property "Reference" "#PWR085"
 			(at 175.26 96.52 0)
 			(hide yes)
@@
 			(project "e-foc"
 				(path "/34e5c7b2-bc7d-4136-97dd-86505a14228c/6cd2b0a0-683f-4196-92a9-4a51f926d77e"
-					(reference "#PWR075")
+					(reference "#PWR085")
 					(unit 1)
 				)
@@
 		(dnp no)
 		(fields_autoplaced yes)
-		(property "Reference" "#PWR072"
+		(property "Reference" "#PWR082"
 			(at 146.05 73.66 0)
 			(hide yes)
@@
 			(project "e-foc"
 				(path "/34e5c7b2-bc7d-4136-97dd-86505a14228c/6cd2b0a0-683f-4196-92a9-4a51f926d77e"
-					(reference "#PWR072")
-					(unit 1)
-				)
+					(reference "#PWR082")
+					(unit 1)
+				)
