File: hardware/e-foc.kicad_sch (KiCad schematic)
At the start: 0 parts

Commit message: refactor structure
Other:
- sheet adc-conditioner: file adc-conditioner.kicad_sch -> schematic/adc-conditioner.kicad_sch
- sheet can-bus: file can-bus.kicad_sch -> schematic/can-bus.kicad_sch
- sheet driver: file driver.kicad_sch -> schematic/driver.kicad_sch
- sheet eeprom-mem: file eeprom-mem.kicad_sch -> schematic/eeprom-mem.kicad_sch
- sheet flash-mem: file flash-mem.kicad_sch -> schematic/flash-mem.kicad_sch
- sheet microcontroller-connector: file microcontroller-connector.kicad_sch -> schematic/microcontroller-connector.kicad_sch
- sheet power-supply: file untitled.kicad_sch -> schematic/untitled.kicad_sch
- sheet serial-com: file serial-com.kicad_sch -> schematic/serial-com.kicad_sch
Changed lines of the file:
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@@
 			)
 		)
-		(property "Sheetfile" "driver.kicad_sch"
+		(property "Sheetfile" "schematic/driver.kicad_sch"
 			(at 63.5 79.3246 0)
 			(show_name yes)
@@
 			)
 		)
-		(property "Sheetfile" "microcontroller-connector.kicad_sch"
+		(property "Sheetfile" "schematic/microcontroller-connector.kicad_sch"
 			(at 109.22 123.7746 0)
 			(show_name no)
@@
 			)
 		)
-		(property "Sheetfile" "flash-mem.kicad_sch"
+		(property "Sheetfile" "schematic/flash-mem.kicad_sch"
 			(at 187.96 141.5546 0)
 			(show_name yes)
@@
 			)
 		)
-		(property "Sheetfile" "adc-conditioner.kicad_sch"
+		(property "Sheetfile" "schematic/adc-conditioner.kicad_sch"
 			(at 50.8 158.0646 0)
 			(show_name yes)
@@
 			)
 		)
-		(property "Sheetfile" "eeprom-mem.kicad_sch"
+		(property "Sheetfile" "schematic/eeprom-mem.kicad_sch"
 			(at 187.96 103.4546 0)
 			(show_name yes)
@@
 			)
 		)
-		(property "Sheetfile" "untitled.kicad_sch"
+		(property "Sheetfile" "schematic/untitled.kicad_sch"
 			(at 114.3 47.5746 0)
 			(show_name no)
@@
 			)
 		)
-		(property "Sheetfile" "serial-com.kicad_sch"
+		(property "Sheetfile" "schematic/serial-com.kicad_sch"
 			(at 189.23 56.4646 0)
 			(show_name yes)
@@
 			)
 		)
-		(property "Sheetfile" "can-bus.kicad_sch"
+		(property "Sheetfile" "schematic/can-bus.kicad_sch"
 			(at 50.8 125.0446 0)
 			(show_name yes)

Commit message: schematic finished
Other:
- removed sheet serial-com
- sheet adc-conditioner ports: added CUR_A, CUR_A_H, CUR_A_L, CUR_B, CUR_B_L, CUR_C, CUR_C_H, CUR_C_L, CUR_TOTAL, CUR_TOTAL_H, CUR_TOTAL_L, CUR­_B_H, VOLT_TOTAL; removed none
- sheet can-bus ports: added CAN_RX, CAN_TX; removed none
- sheet driver ports: added CUR_A_H, CUR_A_L, CUR_B_H, CUR_B_L, CUR_C_H, CUR_C_L, CUR_TOTAL_H, CUR_TOTAL_L, PWM_A_H, PWM_A_L, PWM_B_H, PWM_B_L, PWM_C_H, PWM_C_L; removed none
- sheet eeprom-mem ports: added I2C_SCL, I2C_SDA; removed none
- sheet flash-mem ports: added SPI_CS, SPI_MISO, SPI_MOSI, SPI_SCK; removed none
- sheet microcontroller-connector ports: added CAN_RX, CAN_TX, CUR_A, CUR_B, CUR_C, CUR_TOTAL, I2C_SCL, I2C_SDA, POWER_GOOD, PWM_A_H, PWM_A_L, PWM_B_H, PWM_B_L, PWM_C_H, PWM_C_L, SPI_CS_FLASH, SPI_MISO, SPI_MOSI, SPI_SCK, VOLT_TOTAL; removed none
- sheet power-supply ports: added POWER_GOOD; removed none

Commit message: pcb improvements
Parts:
- added H1, H2, H3, H4: MountingHole, MountingHole:MountingHole_3.2mm_M3_DIN965_Pad_TopBottom, symbol Mechanical:MountingHole
Other:
- added sheet encoder (encoder.kicad_sch)
- sheet adc-conditioner ports: added CUR_A_N, CUR_A_P, CUR_B_N, CUR_C_N, CUR_C_P, CUR_TOTAL_N, CUR_TOTAL_P, CUR­_B_P; removed CUR_A_H, CUR_A_L, CUR_B_L, CUR_C_H, CUR_C_L, CUR_TOTAL_H, CUR_TOTAL_L, CUR­_B_H
- sheet driver ports: added CUR_A_N, CUR_A_P, CUR_B_N, CUR_B_P, CUR_C_N, CUR_C_P, CUR_TOTAL_N, CUR_TOTAL_P; removed CUR_A_H, CUR_A_L, CUR_B_H, CUR_B_L, CUR_C_H, CUR_C_L, CUR_TOTAL_H, CUR_TOTAL_L
- sheet microcontroller-connector ports: added ENC_A, ENC_B, ENC_C; removed none

Commit message: updates
Other:
- sheet encoder: file encoder.kicad_sch -> schematic/encoder.kicad_sch
- sheet power-supply: file schematic/untitled.kicad_sch -> schematic/power-supply.kicad_sch
Changed lines of the file:
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@@
 			)
 		)
-		(property "Sheetfile" "encoder.kicad_sch"
+		(property "Sheetfile" "schematic/encoder.kicad_sch"
 			(at 220.98 92.0246 0)
 			(show_name no)
@@
 			)
 		)
-		(property "Sheetfile" "schematic/untitled.kicad_sch"
+		(property "Sheetfile" "schematic/power-supply.kicad_sch"
 			(at 104.14 97.1046 0)
 			(show_name no)
