File: hardware/e-foc.kicad_pcb (KiCad board)
At the start: 4 copper layers, 89.4 x 66.9 mm, 186 parts, among them J1 Screw_Terminal_01x02, J2 Screw_Terminal_01x03, J3 Screw_Terminal_01x02, J4 Conn_01x05_Pin, J5 Conn_01x03, J6 Conn_02x12_Odd_Even, J7 Conn_02x06_Odd_Even, Q1 CSD88537ND, Q2 CSD88537ND, Q3 CSD88537ND, Q4 BC847, Q5 BC847, Q6 BC847, SW1 SW_DIP_x03, U1 LM5164DDA, U10 W25Q32JVSS, U2 LM317_SOT-223, U3 AMS1117-3.3, U4 FAN7888, U5 TLV9064, U6 TLV9062, U7 SN65HVD230, U8 74LVC14, U9 24LC04

Commit message: board finished
Parts:
- NT1: moved to B.Cu
- U1: footprint Package_SO:HSOP-8-1EP_3.9x4.9mm_P1.27mm_EP2.41x3.1mm_ThermalVias -> Package_SO:HSOP-8-1EP_3.9x4.9mm_P1.27mm_EP2.41x3.1mm
- moved TP3 19.5 mm to (214.5, 111.0)
- moved NT1 17.2 mm to (197.0, 97.5)
- moved R29 4.00 mm to (219.0, 85.0)
- moved C16 2.00 mm to (219.0, 87.0)
- moved R30 2.00 mm to (219.0, 89.0)
Routing:
- net Vdrive: track 48.7 -> 83.8 mm
- net GNDPWR: track 103.4 -> 131.7 mm
- net Net-(J6-Pin_14): track 9.40 -> 32.3 mm, vias 0 -> 2
- net /adc-conditioner/VOLT_TOTAL: track 76.9 -> 65.0 mm, vias 1 -> 3
- net +3.3V: track 124.2 -> 134.0 mm, vias 43 -> 52
- net GND: track 287.9 -> 281.2 mm, vias 48 -> 76
- net /flash-mem/SPI_CS: track 28.5 -> 26.3 mm
- net Net-(U10-~{WP}/IO_{2}): track 12.5 -> 14.7 mm
- net Net-(J6-Pin_12): track 35.3 -> 33.4 mm
- net /adc-conditioner/CUR_TOTAL_P: track 34.2 -> 32.4 mm
- net /adc-conditioner/CUR_C_N: track 33.0 -> 34.6 mm
- net /adc-conditioner/CUR_TOTAL_N: track 37.0 -> 35.6 mm
- net Net-(U9-A1): track 8.99 -> 10.4 mm
- net Net-(J4-Pin_5): track 77.5 -> 78.4 mm
- net Net-(J4-Pin_4): track 77.2 -> 78.1 mm
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- added copper zone on F.Cu, net Net-(NT2-Pad1)
- added copper zone on F.Cu, net Net-(NT4-Pad1)
- added copper zone on F.Cu, net Net-(NT8-Pad1)

Commit message: updates
Routing:
- net Net-(J5-Pin_2): track 0.00 -> 68.2 mm
- net Net-(J5-Pin_3): track 0.00 -> 66.9 mm
Other:
- copper layers 4 -> 2

Commit message: updates
Parts:
- D1: value SMCJ60CA -> SMCJ51A
- J3: value Screw_Terminal_01x02 -> Screw_Terminal_01x03; footprint TerminalBlock_TE-Connectivity:TerminalBlock_TE_282834-2_1x02_P2.54mm_Horizontal -> TerminalBlock:TerminalBlock_Xinya_XY308-2.54-3P_1x03_P2.54mm_Horizontal
- R1: value 187k -> 124k
- R2: value 194k -> 280k
- R3: value 787k -> 576k
- moved J3 0.41 mm to (245.0, 141.3)
- renumbered R81 to R77, R82 to R78, R80 to R79, R79 to R80, R78 to R81, R77 to R82
Connections:
- net +20V renamed +15V
- D6 pad 1: Net-(J3-Pin_2) -> Net-(J3-Pin_3)
- J3 pad 2: Net-(J3-Pin_2) -> GND
- R51 pad 2: Net-(J3-Pin_2) -> Net-(J3-Pin_3)
- U7 pad 6: Net-(J3-Pin_2) -> Net-(J3-Pin_3)
Routing:
- net Net-(J3-Pin_3): track 0.00 -> 21.1 mm
- net Net-(J3-Pin_2): track 17.5 -> 0.00 mm
- net GND: track 281.2 -> 266.2 mm, vias 76 -> 90
- net Net-(J3-Pin_1): track 12.0 -> 11.5 mm

Commit message: .\.claude\
Parts:
- moved H3 0.72 mm to (255.2, 141.0)
- moved H4 0.72 mm to (255.2, 84.0)
Routing:
- net GND: track 266.2 -> 251.3 mm
- net GNDPWR: track 131.7 -> 120.2 mm, vias 11 -> 71
- net +5V: track 207.1 -> 204.2 mm
Other:
- board text added: "+5V"
- board text added: "+V (55 Vdc max)"
- board text added: "A"
- board text added: "B"
- board text added: "C"
- board text added: "GND"
- board text added: "Z"
- board text added: "e-FOC v1.0"
