File: hardware/e-foc/schematic/flash-mem.kicad_sch (KiCad schematic)
At the start: 6 parts, among them U2 W25Q32JVSS

Commit message: chore: add release please action (#1)
* add release please action

* refactor structure

* schematic finished

* pcb improvements

* board finished

* updates

* updates

* .\.claude\

* updates

* reorganize project

* fix ci

* fix ci

* fix(ci): disable kicad-bot bom/diff (not implemented in v0.1.3)

verify (ERC/DRC) passes, but run-bom-check and run-diff exit 2 with
"not available in this build yet (Phase 2/3)". Keep run-verify only.

Co-Authored-By: Claude Opus 4.8 <noreply@anthropic.com>

* feat(ci): visual schematic/PCB diff on pull requests

kicad-bot's diff phase isn't available in v0.1.x, so render PR head vs base
with kicad-cli and produce a red/green overlay (added/removed) per board via
Pillow — no KiAuto/GUI automation. New scripts/visual_diff.py + a matrix
kicad-diff.yml that uploads the diff images as a per-board artifact.

Co-Authored-By: Claude Opus 4.8 <noreply@anthropic.com>

* fix(erc): ignore power_pin_not_driven instead of per-instance exclusions

Both boards are powered through a connector, so power_pin_not_driven is an
expected false-positive. It was suppressed via GUI per-instance exclusions
(hashed by coordinates/UUIDs), which don't survive a different KiCad patch or
the PR merge commit in CI -> the violations resurfaced as ERC errors and
failed verify (e.g. tiva: 4 errors). Set the rule severity to "ignore" in
each .kicad_pro: deterministic, committed, version-independent. 0 ERC errors
on both boards now.

Co-Authored-By: Claude Opus 4.8 <noreply@anthropic.com>

---------

Co-authored-by: Claude Opus 4.8 <noreply@anthropic.com>
Parts:
- C36: renamed from C?; footprint (none) -> Capacitor_SMD:C_0805_2012Metric_Pad1.18x1.45mm_HandSolder
- gave numbers to parts that had none: 4
- renumbered U2 to U10
Changed lines of the file:
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@@
 		)
 	)
-	(global_label "SPI_MISO"
-		(shape input)
+	(hierarchical_label "SPI_MISO"
+		(shape output)
 		(at 118.11 82.55 180)
-		(fields_autoplaced yes)
 		(effects
 			(font
@@
 			(justify right)
 		)
-		(property "Intersheetrefs" "${INTERSHEET_REFS}"
-			(at 106.4767 82.55 0)
-			(hide yes)
-			(show_name no)
-			(do_not_autoplace no)
-			(effects
-				(font
-					(size 1.27 1.27)
-				)
-				(justify right)
-			)
-		)
-	)
-	(global_label "SPI_CS"
-		(shape input)
-		(at 118.11 77.47 180)
-		(fields_autoplaced yes)
+	)
+	(hierarchical_label "SPI_MOSI"
+		(shape output)
+		(at 118.11 85.09 180)
 		(effects
 			(font
@@
 			(justify right)
 		)
-		(property "Intersheetrefs" "${INTERSHEET_REFS}"
-			(at 108.5934 77.47 0)
-			(hide yes)
-			(show_name no)
-			(do_not_autoplace no)
-			(effects
-				(font
-					(size 1.27 1.27)
-				)
-				(justify right)
-			)
-		)
-	)
-	(global_label "SPI_SCK"
-		(shape input)
-		(at 118.11 80.01 180)
-		(fields_autoplaced yes)
+	)
+	(hierarchical_label "SPI_CS"
+		(shape output)
+		(at 118.11 77.47 180)
 		(effects
 			(font
@@
 			(justify right)
 		)
-		(property "Intersheetrefs" "${INTERSHEET_REFS}"
-			(at 107.3234 80.01 0)
-			(hide yes)
-			(show_name no)
-			(do_not_autoplace no)
-			(effects
-				(font
-					(size 1.27 1.27)
-				)
-				(justify right)
-			)
-		)
-	)
-	(global_label "SPI_MOSI"
-		(shape input)
-		(at 118.11 85.09 180)
-		(fields_autoplaced yes)
+	)
+	(hierarchical_label "SPI_SCK"
+		(shape output)
+		(at 118.11 80.01 180)
 		(effects
 			(font
@@
 			(justify right)
 		)
-		(property "Intersheetrefs" "${INTERSHEET_REFS}"
-			(at 106.4767 85.09 0)
-			(hide yes)
-			(show_name no)
-			(do_not_autoplace no)
-			(effects
-				(font
-					(size 1.27 1.27)
-				)
-				(justify right)
-			)
-		)
 	)
 	(symbol
@@
 		(in_pos_files yes)
 		(dnp no)
-		(property "Reference" "R?"
-			(at 124.968 95.25 90)
+		(property "Reference" "R71"
+			(at 123.698 94.996 90)
 			(show_name no)
 			(do_not_autoplace no)
@@
 			(project "e-foc"
 				(path "/34e5c7b2-bc7d-4136-97dd-86505a14228c/6cd2b0a0-683f-4196-92a9-4a51f926d77e"
-					(reference "R?")
+					(reference "R71")
 					(unit 1)
 				)
@@
 		(dnp no)
 		(fields_autoplaced yes)
-		(property "Reference" "#PWR045"
+		(property "Reference" "#PWR084"
 			(at 146.05 105.41 0)
 			(hide yes)
@@
 			(project "e-foc"
 				(path "/34e5c7b2-bc7d-4136-97dd-86505a14228c/6cd2b0a0-683f-4196-92a9-4a51f926d77e"
-					(reference "#PWR045")
+					(reference "#PWR084")
 					(unit 1)
 				)
@@
 		(in_pos_files yes)
 		(dnp no)
-		(property "Reference" "R?"
+		(property "Reference" "R72"
 			(at 135.89 71.1199 0)
 			(show_name no)
@@
 			(project "e-foc"
 				(path "/34e5c7b2-bc7d-4136-97dd-86505a14228c/6cd2b0a0-683f-4196-92a9-4a51f926d77e"
-					(reference "R?")
+					(reference "R72")
 					(unit 1)
 				)
@@
 		(dnp no)
 		(fields_autoplaced yes)
-		(property "Reference" "#PWR049"
+		(property "Reference" "#PWR085"
 			(at 175.26 83.82 0)
 			(hide yes)
@@
 			(project "e-foc"
 				(path "/34e5c7b2-bc7d-4136-97dd-86505a14228c/6cd2b0a0-683f-4196-92a9-4a51f926d77e"
-					(reference "#PWR049")
+					(reference "#PWR085")
 					(unit 1)
 				)
@@
 		(dnp no)
 		(fields_autoplaced yes)
-		(property "Reference" "#PWR046"
+		(property "Reference" "#PWR082"
 			(at 133.35 69.85 0)
 			(hide yes)
@@
 			(project "e-foc"
 				(path "/34e5c7b2-bc7d-4136-97dd-86505a14228c/6cd2b0a0-683f-4196-92a9-4a51f926d77e"
-					(reference "#PWR046")
+					(reference "#PWR082")
 					(unit 1)
 				)
@@
 		(in_pos_files yes)
 		(dnp no)
-		(property "Reference" "R?"
-			(at 124.968 90.17 90)
+		(property "Reference" "R70"
+			(at 123.444 90.17 90)
 			(show_name no)
 			(do_not_autoplace no)
@@
 			(project "e-foc"
 				(path "/34e5c7b2-bc7d-4136-97dd-86505a14228c/6cd2b0a0-683f-4196-92a9-4a51f926d77e"
-					(reference "R?")
+					(reference "R70")
 					(unit 1)
 				)
@@
 		(in_pos_files yes)
 		(dnp no)
-		(property "Reference" "C?"
+		(property "Reference" "C36"
 			(at 179.07 83.8199 0)
 			(show_name no)
@@
 			)
 		)
-		(property "Footprint" ""
+		(property "Footprint" "Capacitor_SMD:C_0805_2012Metric_Pad1.18x1.45mm_HandSolder"
 			(at 176.2252 88.9 0)
 			(hide yes)
@@
 			(project "e-foc"
 				(path "/34e5c7b2-bc7d-4136-97dd-86505a14228c/6cd2b0a0-683f-4196-92a9-4a51f926d77e"
-					(reference "C?")
+					(reference "C36")
 					(unit 1)
 				)
@@
 		(dnp no)
 		(fields_autoplaced yes)
-		(property "Reference" "#PWR047"
+		(property "Reference" "#PWR081"
 			(at 104.14 88.9 0)
 			(hide yes)
@@
 			(project "e-foc"
 				(path "/34e5c7b2-bc7d-4136-97dd-86505a14228c/6cd2b0a0-683f-4196-92a9-4a51f926d77e"
-					(reference "#PWR047")
+					(reference "#PWR081")
 					(unit 1)
 				)
@@
 		(dnp no)
 		(fields_autoplaced yes)
-		(property "Reference" "U2"
+		(property "Reference" "U10"
 			(at 157.48 83.8199 0)
 			(show_name no)
@@
 			(project "e-foc"
 				(path "/34e5c7b2-bc7d-4136-97dd-86505a14228c/6cd2b0a0-683f-4196-92a9-4a51f926d77e"
-					(reference "U2")
+					(reference "U10")
 					(unit 1)
 				)
@@
 		(in_pos_files yes)
 		(dnp no)
-		(property "Reference" "R?"
-			(at 122.936 75.692 90)
+		(property "Reference" "R69"
+			(at 121.92 75.692 90)
 			(show_name no)
 			(do_not_autoplace no)
@@
 			(project "e-foc"
 				(path "/34e5c7b2-bc7d-4136-97dd-86505a14228c/6cd2b0a0-683f-4196-92a9-4a51f926d77e"
-					(reference "R?")
+					(reference "R69")
 					(unit 1)
 				)
@@
 		(dnp no)
 		(fields_autoplaced yes)
-		(property "Reference" "#PWR048"
+		(property "Reference" "#PWR086"
 			(at 175.26 96.52 0)
 			(hide yes)
@@
 			(project "e-foc"
 				(path "/34e5c7b2-bc7d-4136-97dd-86505a14228c/6cd2b0a0-683f-4196-92a9-4a51f926d77e"
-					(reference "#PWR048")
+					(reference "#PWR086")
 					(unit 1)
 				)
@@
 		(dnp no)
 		(fields_autoplaced yes)
-		(property "Reference" "#PWR044"
+		(property "Reference" "#PWR083"
 			(at 146.05 73.66 0)
 			(hide yes)
@@
 			(project "e-foc"
 				(path "/34e5c7b2-bc7d-4136-97dd-86505a14228c/6cd2b0a0-683f-4196-92a9-4a51f926d77e"
-					(reference "#PWR044")
-					(unit 1)
-				)
+					(reference "#PWR083")
+					(unit 1)
+				)
